File: board/comms 2.brd (EAGLE design)
At the start: 88.6 x 50.8 mm, 23 parts, among them CON1 ISP, CON3 1X03, CON6 TE_2-PIN, J2 4-644694-4, U1 ESP-WROOM-02D, U2 ATMEGA328PB-AN

Commit message: Update board files
Connections:
- net BE: now also U2.2; no longer U2.30
- net CMD_DATA_IN: now also U2.31; no longer U2.3
- net CMD_DATA_OUT: now also U2.30; no longer U2.2
- net EX: now also U2.3; no longer U2.31
- net V_3.3: now also CON1.2
- net V_BATT: no longer CON1.2
Routing:
- net V_BATT: track 104.7 -> 21.8 mm
- net V_3.3: track 217.5 -> 242.4 mm
- net BE: track 6.98 -> 11.7 mm, vias 0 -> 1
- net EX: track 8.58 -> 12.1 mm, vias 0 -> 1
- net CMD_DATA_OUT: track 14.5 -> 17.5 mm, vias 0 -> 1
- net CMD_DATA_IN: track 17.4 -> 19.3 mm, vias 0 -> 1
Changed lines of the file:
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@@
 <drawing>
 <settings>
-<setting alwaysvectorfont="yes"/>
+<setting alwaysvectorfont="no"/>
 <setting verticaltext="up"/>
 </settings>
@@
 </signal>
 <signal name="V_BATT">
-<contactref element="CON1" pad="2"/>
 <contactref element="C3" pad="1"/>
 <contactref element="VR1" pad="3"/>
@@
 <wire x1="9.121" y1="53.594" x2="10.137" y2="54.61" width="1.27" layer="1"/>
 <wire x1="10.137" y1="54.61" x2="12.192" y2="54.61" width="1.27" layer="1"/>
-<wire x1="45.72" y1="73.66" x2="5.08" y2="73.66" width="1.27" layer="1"/>
-<wire x1="5.08" y1="73.66" x2="1.651" y2="70.231" width="1.27" layer="1"/>
-<wire x1="10.13" y1="40.17" x2="13.94" y2="40.17" width="1.27" layer="1"/>
-<wire x1="10.13" y1="40.17" x2="1.651" y2="48.649" width="1.27" layer="1"/>
-<wire x1="1.651" y1="70.231" x2="1.651" y2="48.649" width="1.27" layer="1"/>
 <wire x1="12.192" y1="55.118" x2="12.192" y2="55.252" width="1.27" layer="1"/>
 <wire x1="14.014296875" y1="53.295703125" x2="12.192" y2="55.118" width="1.27" layer="1"/>
@@
 <wire x1="10.16" y1="66.89284375" x2="8.4962" y2="68.55664375" width="0.8128" layer="1"/>
 <wire x1="22.76915625" y1="71.755" x2="23.576578125" y2="70.947578125" width="0.8128" layer="1"/>
-<wire x1="10.63184375" y1="71.755" x2="22.76915625" y2="71.755" width="0.8128" layer="1"/>
+<wire x1="10.63184375" y1="71.755" x2="21.59" y2="71.755" width="0.8128" layer="1"/>
+<wire x1="21.59" y1="71.755" x2="22.76915625" y2="71.755" width="0.8128" layer="1"/>
 <wire x1="39" y1="60.09" x2="32.62" y2="60.09" width="0.4064" layer="1"/>
 <wire x1="32.62" y1="60.09" x2="31.75" y2="60.96" width="0.4064" layer="1"/>
@@
 <wire x1="77.955" y1="73.66" x2="80.01" y2="73.66" width="0.8128" layer="1"/>
 <wire x1="80.795" y1="77.47" x2="80.795" y2="73.66" width="0.8128" layer="1"/>
+<contactref element="CON1" pad="2"/>
+<wire x1="21.59" y1="71.755" x2="23.495" y2="73.66" width="0.508" layer="1"/>
+<wire x1="23.495" y1="73.66" x2="45.72" y2="73.66" width="0.508" layer="1"/>
 <wire x1="80.01" y1="73.66" x2="80.795" y2="73.66" width="0" layer="19" extent="1-1"/>
 </signal>
@@
 <signal name="BE">
 <contactref element="J2" pad="1"/>
-<contactref element="U2" pad="30"/>
-<wire x1="37.719" y1="69.088" x2="41.98" y2="64.827" width="0.3048" layer="1"/>
-<wire x1="41.98" y1="64.827" x2="41.98" y2="63.87" width="0.3048" layer="1"/>
+<contactref element="U2" pad="2"/>
+<wire x1="39" y1="61.69" x2="41.37" y2="61.69" width="0.3048" layer="1"/>
+<wire x1="41.37" y1="61.69" x2="41.91" y2="62.23" width="0.3048" layer="1"/>
+<via x="41.91" y="62.23" extent="1-16" drill="0.35"/>
+<wire x1="41.91" y1="62.23" x2="40.132" y2="64.008" width="0.3048" layer="16"/>
+<wire x1="40.132" y1="66.167" x2="37.719" y2="68.58" width="0.3048" layer="16"/>
+<wire x1="37.719" y1="69.088" x2="37.719" y2="68.58" width="0.3048" layer="16"/>
+<wire x1="40.132" y1="64.008" x2="40.132" y2="66.167" width="0.3048" layer="16"/>
 </signal>
 <signal name="EX">
 <contactref element="J2" pad="2"/>
-<contactref element="U2" pad="31"/>
-<wire x1="35.179" y1="69.088" x2="36.957" y2="67.31" width="0.3048" layer="1"/>
-<wire x1="38.44605" y1="67.31" x2="41.18" y2="64.57605" width="0.3048" layer="1"/>
-<wire x1="41.18" y1="64.57605" x2="41.18" y2="63.87" width="0.3048" layer="1"/>
-<wire x1="36.957" y1="67.31" x2="38.44605" y2="67.31" width="0.3048" layer="1"/>
+<contactref element="U2" pad="3"/>
+<wire x1="39" y1="60.89" x2="39.07" y2="60.96" width="0.3048" layer="1"/>
+<wire x1="39.07" y1="60.96" x2="40.64" y2="60.96" width="0.3048" layer="1"/>
+<via x="40.64" y="60.96" extent="1-16" drill="0.35"/>
+<wire x1="40.64" y1="60.96" x2="40.64" y2="62.85341875" width="0.3048" layer="16"/>
+<wire x1="40.64" y1="62.85341875" x2="39.1668" y2="64.32661875" width="0.3048" layer="16"/>
+<wire x1="39.1668" y1="65.1002" x2="35.179" y2="69.088" width="0.3048" layer="16"/>
+<wire x1="39.1668" y1="64.32661875" x2="39.1668" y2="65.1002" width="0.3048" layer="16"/>
 </signal>
 <signal name="CRESP">
@@
 <signal name="CMD_DATA_OUT">
 <contactref element="J2" pad="5"/>
-<contactref element="U2" pad="2"/>
-<wire x1="27.559" y1="69.088" x2="34.957" y2="61.69" width="0.3048" layer="1"/>
-<wire x1="34.957" y1="61.69" x2="39" y2="61.69" width="0.3048" layer="1"/>
+<contactref element="U2" pad="30"/>
+<via x="35.306" y="67.485" extent="1-16" drill="0.35"/>
+<wire x1="41.98" y1="63.87" x2="42.0138" y2="63.9038" width="0.3048" layer="1"/>
+<wire x1="42.0138" y1="65.31278125" x2="42.0138" y2="63.9038" width="0.3048" layer="1"/>
+<wire x1="42.0138" y1="65.31278125" x2="39.84158125" y2="67.485" width="0.3048" layer="1"/>
+<wire x1="39.84158125" y1="67.485" x2="35.306" y2="67.485" width="0.3048" layer="1"/>
+<wire x1="35.306" y1="67.485" x2="29.162" y2="67.485" width="0.3048" layer="16"/>
+<wire x1="29.162" y1="67.485" x2="27.559" y2="69.088" width="0.3048" layer="16"/>
 </signal>
 <signal name="CMD_DATA_IN">
 <contactref element="J2" pad="6"/>
-<contactref element="U2" pad="3"/>
-<wire x1="28.829" y1="66.548" x2="27.559" y2="66.548" width="0.3048" layer="1"/>
-<wire x1="25.019" y1="69.088" x2="27.559" y2="66.548" width="0.3048" layer="1"/>
-<wire x1="34.487" y1="60.89" x2="28.829" y2="66.548" width="0.3048" layer="1"/>
-<wire x1="34.487" y1="60.89" x2="39" y2="60.89" width="0.3048" layer="1"/>
+<contactref element="U2" pad="31"/>
+<wire x1="41.18" y1="63.87" x2="41.18" y2="65.5" width="0.3048" layer="1"/>
+<wire x1="39.878" y1="66.802" x2="36.195" y2="66.802" width="0.3048" layer="1"/>
+<via x="36.195" y="66.802" extent="1-16" drill="0.35"/>
+<wire x1="36.195" y1="66.802" x2="27.305" y2="66.802" width="0.3048" layer="16"/>
+<wire x1="27.305" y1="66.802" x2="25.019" y2="69.088" width="0.3048" layer="16"/>
+<wire x1="41.18" y1="65.5" x2="39.878" y2="66.802" width="0.3048" layer="1"/>
 </signal>
 <signal name="PWR_DOWN">
