File: board/comms 2.sch (EAGLE design)
At the start: 23 parts, among them CON1 ISP, CON3 1X03, CON6 TE_2-PIN, J2 4-644694-4, U1 ESP-WROOM-02D, U2 ATMEGA328PB-AN

Commit message: Update board files
Connections:
- net BE: now also U2.PD4/XCK0/T0/PTCXY; no longer U2.PD0/PTCXY/OC3A/RXD0
- net CMD_DATA_IN: now also U2.PD1/PTCXY/OC4A/TXD0; no longer U2.PE0/SDA1/ICP4/ACO/PTCXY
- net CMD_DATA_OUT: now also U2.PD0/PTCXY/OC3A/RXD0; no longer U2.PD4/XCK0/T0/PTCXY
- net EX: now also U2.PE0/SDA1/ICP4/ACO/PTCXY; no longer U2.PD1/PTCXY/OC4A/TXD0
- net V_3.3: now also CON1.2
- net V_BATT: no longer CON1.2
Changed lines of the file:
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@@
 <net name="V_BATT" class="0">
-<segment>
-<pinref part="CON1" gate="G$1" pin="2"/>
-<wire x1="-132.08" y1="173.99" x2="-127" y2="173.99" width="0.1524" layer="91"/>
-<label x="-129.54" y="176.53" size="1.778" layer="95"/>
-</segment>
 <segment>
 <wire x1="-180.34" y1="59.69" x2="-170.18" y2="59.69" width="0.1524" layer="91"/>
@@
 <label x="-5.08" y="182.88" size="1.778" layer="95"/>
 </segment>
+<segment>
+<pinref part="CON1" gate="G$1" pin="2"/>
+<wire x1="-132.08" y1="173.99" x2="-127" y2="173.99" width="0.1524" layer="91"/>
+<label x="-129.54" y="176.53" size="1.778" layer="95"/>
+</segment>
 </net>
 <net name="TXD_WIFI" class="0">
@@
 </segment>
 <segment>
+<pinref part="U2" gate="G$1" pin="PD4/XCK0/T0/PTCXY"/>
+<wire x1="-104.648" y1="134.62" x2="-99.06" y2="134.62" width="0.1524" layer="91"/>
+<label x="-99.06" y="134.62" size="1.778" layer="95"/>
+</segment>
+</net>
+<net name="EX" class="0">
+<segment>
+<pinref part="J2" gate="G$1" pin="2"/>
+<wire x1="40.64" y1="76.2" x2="35.56" y2="76.2" width="0.1524" layer="91"/>
+<label x="30.48" y="76.2" size="1.778" layer="95"/>
+</segment>
+<segment>
+<pinref part="U2" gate="G$1" pin="PE0/SDA1/ICP4/ACO/PTCXY"/>
+<wire x1="-104.648" y1="114.3" x2="-99.06" y2="114.3" width="0.1524" layer="91"/>
+<label x="-99.06" y="114.3" size="1.778" layer="95"/>
+</segment>
+</net>
+<net name="CRESP" class="0">
+<segment>
+<pinref part="J2" gate="G$1" pin="3"/>
+<wire x1="40.64" y1="73.66" x2="35.56" y2="73.66" width="0.1524" layer="91"/>
+<label x="27.94" y="73.66" size="1.778" layer="95"/>
+</segment>
+<segment>
+<pinref part="U2" gate="G$1" pin="PD2/PTCXY/INT0/OC3B/OC4B"/>
+<wire x1="-104.648" y1="139.7" x2="-99.314" y2="139.7" width="0.1524" layer="91"/>
+<label x="-99.06" y="139.7" size="1.778" layer="95"/>
+</segment>
+</net>
+<net name="PB" class="0">
+<segment>
+<pinref part="J2" gate="G$1" pin="4"/>
+<wire x1="40.64" y1="71.12" x2="35.56" y2="71.12" width="0.1524" layer="91"/>
+<label x="30.48" y="71.12" size="1.778" layer="95"/>
+</segment>
+<segment>
+<pinref part="U2" gate="G$1" pin="PD3/OC2B/INT1/PTCXY"/>
+<wire x1="-104.648" y1="137.16" x2="-99.568" y2="137.16" width="0.1524" layer="91"/>
+<label x="-99.06" y="137.16" size="1.778" layer="95"/>
+</segment>
+</net>
+<net name="CMD_DATA_OUT" class="0">
+<segment>
+<pinref part="J2" gate="G$1" pin="5"/>
+<wire x1="40.64" y1="68.58" x2="35.56" y2="68.58" width="0.1524" layer="91"/>
+<label x="15.24" y="68.58" size="1.778" layer="95"/>
+</segment>
+<segment>
 <pinref part="U2" gate="G$1" pin="PD0/PTCXY/OC3A/RXD0"/>
 <wire x1="-104.648" y1="144.78" x2="-99.568" y2="144.78" width="0.1524" layer="91"/>
@@
 </segment>
 </net>
-<net name="EX" class="0">
-<segment>
-<pinref part="J2" gate="G$1" pin="2"/>
-<wire x1="40.64" y1="76.2" x2="35.56" y2="76.2" width="0.1524" layer="91"/>
-<label x="30.48" y="76.2" size="1.778" layer="95"/>
+<net name="CMD_DATA_IN" class="0">
+<segment>
+<pinref part="J2" gate="G$1" pin="6"/>
+<wire x1="40.64" y1="66.04" x2="35.56" y2="66.04" width="0.1524" layer="91"/>
+<label x="17.78" y="66.04" size="1.778" layer="95"/>
 </segment>
 <segment>
@@
 </segment>
 </net>
-<net name="CRESP" class="0">
-<segment>
-<pinref part="J2" gate="G$1" pin="3"/>
-<wire x1="40.64" y1="73.66" x2="35.56" y2="73.66" width="0.1524" layer="91"/>
-<label x="27.94" y="73.66" size="1.778" layer="95"/>
-</segment>
-<segment>
-<pinref part="U2" gate="G$1" pin="PD2/PTCXY/INT0/OC3B/OC4B"/>
-<wire x1="-104.648" y1="139.7" x2="-99.314" y2="139.7" width="0.1524" layer="91"/>
-<label x="-99.06" y="139.7" size="1.778" layer="95"/>
-</segment>
-</net>
-<net name="PB" class="0">
-<segment>
-<pinref part="J2" gate="G$1" pin="4"/>
-<wire x1="40.64" y1="71.12" x2="35.56" y2="71.12" width="0.1524" layer="91"/>
-<label x="30.48" y="71.12" size="1.778" layer="95"/>
-</segment>
-<segment>
-<pinref part="U2" gate="G$1" pin="PD3/OC2B/INT1/PTCXY"/>
-<wire x1="-104.648" y1="137.16" x2="-99.568" y2="137.16" width="0.1524" layer="91"/>
-<label x="-99.06" y="137.16" size="1.778" layer="95"/>
-</segment>
-</net>
-<net name="CMD_DATA_OUT" class="0">
-<segment>
-<pinref part="J2" gate="G$1" pin="5"/>
-<wire x1="40.64" y1="68.58" x2="35.56" y2="68.58" width="0.1524" layer="91"/>
-<label x="15.24" y="68.58" size="1.778" layer="95"/>
-</segment>
-<segment>
-<pinref part="U2" gate="G$1" pin="PD4/XCK0/T0/PTCXY"/>
-<wire x1="-104.648" y1="134.62" x2="-99.06" y2="134.62" width="0.1524" layer="91"/>
-<label x="-99.06" y="134.62" size="1.778" layer="95"/>
-</segment>
-</net>
-<net name="CMD_DATA_IN" class="0">
-<segment>
-<pinref part="J2" gate="G$1" pin="6"/>
-<wire x1="40.64" y1="66.04" x2="35.56" y2="66.04" width="0.1524" layer="91"/>
-<label x="17.78" y="66.04" size="1.778" layer="95"/>
-</segment>
-<segment>
-<pinref part="U2" gate="G$1" pin="PE0/SDA1/ICP4/ACO/PTCXY"/>
-<wire x1="-104.648" y1="114.3" x2="-99.06" y2="114.3" width="0.1524" layer="91"/>
-<label x="-99.06" y="114.3" size="1.778" layer="95"/>
-</segment>
-</net>
